File: hardware/morse/morse.kicad_sch (KiCad schematic)
At the start: 26 parts, among them J1 Tag-Connect 6P Connector, Q1 SSM3J36FS, U1 ATtiny1617-M

Commit message: Schematic progress
Parts:
- removed LA1: Touch Sensor, symbol Device:Lamp
- added R6, R7: 1k, libraries:Worthington_R_0402, symbol Device:R_Small_US
- added R8: 10k, symbol Device:R_Small_US
- added TS1: XY Touch Pad, libraries:TouchPad_12mm_XY, symbol Device:Lamp_Neon
Connections:
- net +3V0: now also J1.6 (Pin_6), R8.1
- net GND: now also J1.4 (Pin_4); no longer J1.3 (Pin_3)
- net UPDI: now also J1.5 (Pin_5), R8.2; no longer J1.6 (Pin_6)
- net TOUCHY_T: now reaches U1.15 (PB1)
- net TOUCHY_T: now also R7.1
- net TOUCHX_T: now reaches U1.16 (PB0)
- net TOUCHX_T: now also R6.1
- new net TOUCHX: R6.2, TS1.1
- new net TOUCHY: R7.2, TS1.2
